Commit message: First flipper version

File: spider_simulation/src/spider_robot_description/gazebo/spider_robot.gazebo.xacro (robot description, xacro)
@@ -44,11 +44,10 @@
         <odom_publish_frequency>50</odom_publish_frequency>
       </plugin>
-      <!-- Flippers: the four steering joints stand in for flipper pivots.
-           Position control holds them against gravity, which is what the real
-           Teensy PID loop does. -->
-      <xacro:flipper_controller joint="fl_steering_joint" topic="flipper/fl"/>
-      <xacro:flipper_controller joint="fr_steering_joint" topic="flipper/fr"/>
-      <xacro:flipper_controller joint="rl_steering_joint" topic="flipper/rl"/>
-      <xacro:flipper_controller joint="rr_steering_joint" topic="flipper/rr"/>
+      <!-- Position control holds the flippers against gravity, matching the
+           real Teensy PID loop. -->
+      <xacro:flipper_controller joint="fl_flipper_joint" topic="flipper/fl"/>
+      <xacro:flipper_controller joint="fr_flipper_joint" topic="flipper/fr"/>
+      <xacro:flipper_controller joint="rl_flipper_joint" topic="flipper/rl"/>
+      <xacro:flipper_controller joint="rr_flipper_joint" topic="flipper/rr"/>
       <!-- Telemetry source for the Teensy bridge. -->
       <plugin filename="gz-sim-joint-state-publisher-system"

File: spider_simulation/src/spider_robot_description/robots/parts/base/base.urdf.xacro (robot description, xacro)
@@ -2,4 +2,35 @@
 <robot xmlns:xacro="http://ros.org/wiki/xacro">
   <xacro:include filename="$(find spider_robot_description)/robots/parts/base/base.gazebo.xacro"/>
+  <xacro:macro name="main_track_visual" params="side">
+	<!-- Fixed visible track; hidden wheel contacts supply its motion. -->
+	<visual>
+	  <origin xyz="0 ${side * 0.052} -0.010"/>
+	  <geometry>
+		<box size="0.145 0.030 0.047"/>
+	  </geometry>
+	  <material name="track_rubber"/>
+	</visual>
+	<visual>
+	  <origin xyz="0 ${side * 0.052} -0.010"/>
+	  <geometry>
+		<box size="0.108 0.033 0.027"/>
+	  </geometry>
+	  <material name="spider_orange"/>
+	</visual>
+	<visual>
+	  <origin xyz="0.050 ${side * 0.052} -0.010" rpy="1.57079632679 0 0"/>
+	  <geometry>
+		<cylinder radius="0.017" length="0.035"/>
+	  </geometry>
+	  <material name="roller_metal"/>
+	</visual>
+	<visual>
+	  <origin xyz="-0.050 ${side * 0.052} -0.010" rpy="1.57079632679 0 0"/>
+	  <geometry>
+		<cylinder radius="0.017" length="0.035"/>
+	  </geometry>
+	  <material name="roller_metal"/>
+	</visual>
+  </xacro:macro>
   <xacro:macro name="base_v0" params="parent *joint_origin">
 	<joint name="base_link_joint" type="fixed">
@@ -14,4 +45,6 @@
 		</geometry>
 	  </visual>
+	  <xacro:main_track_visual side="1"/>
+	  <xacro:main_track_visual side="-1"/>
 	  <collision>
 		<origin xyz="0 0 0.017"/>

File: spider_simulation/src/spider_robot_description/robots/parts/suspension/suspension.gazebo.xacro (robot description, xacro)
@@ -1,6 +1,6 @@
 <?xml version="1.0"?>
 <robot xmlns:xacro="http://ros.org/wiki/xacro">
-  <xacro:macro name="steering_gazebo_v0" params="prefix">
-	<gazebo reference="${prefix}_steering_link">
+  <xacro:macro name="flipper_gazebo_v0" params="prefix">
+	<gazebo reference="${prefix}_flipper_link">
 	  <selfCollide>false</selfCollide>
       <mu1 value="0.05" />

File: spider_simulation/src/spider_robot_description/robots/parts/suspension/suspension.urdf.xacro (robot description, xacro)
@@ -2,28 +2,54 @@
 <robot xmlns:xacro="http://ros.org/wiki/xacro">
   <xacro:include filename="$(find spider_robot_description)/robots/parts/suspension/suspension.gazebo.xacro"/>
-  <xacro:macro name="steering_v0" params="prefix parent *joint_origin *joint_axis">
-	<joint name="${prefix}_steering_joint" type="revolute">
+  <xacro:macro name="flipper_v0" params="prefix parent direction side *joint_origin *joint_axis">
+	<joint name="${prefix}_flipper_joint" type="revolute">
 	  <xacro:insert_block name="joint_origin"/>
 	  <parent link="${parent}"/>
-	  <child link="${prefix}_steering_link"/>
+	  <child link="${prefix}_flipper_link"/>
           <limit effort="5" velocity="6.28"  lower="-2.1" upper="2.1" />
           <xacro:insert_block name="joint_axis"/>
 	</joint>
-	<link name="${prefix}_steering_link">
+	<link name="${prefix}_flipper_link">
+	  <!-- Rubber belt around the flipper body. -->
 	  <visual>
+		<origin xyz="${direction * 0.045} ${side * 0.020} -0.010"/>
 		<geometry>
-		  <mesh filename="package://spider_robot_description/meshes/DAE/suspension/${prefix}_link.dae"/>
+		  <box size="0.105 0.026 0.034"/>
 		</geometry>
+		<material name="track_rubber"/>
+	  </visual>
+	  <!-- Coloured side plate leaves a dark belt visible around its edge. -->
+	  <visual>
+		<origin xyz="${direction * 0.045} ${side * 0.020} -0.010"/>
+		<geometry>
+		  <box size="0.077 0.029 0.018"/>
+		</geometry>
+		<material name="spider_orange"/>
+	  </visual>
+	  <!-- End rollers make the primitive geometry read as a tracked flipper. -->
+	  <visual>
+		<origin xyz="${direction * 0.010} ${side * 0.020} -0.010" rpy="1.57079632679 0 0"/>
+		<geometry>
+		  <cylinder radius="0.012" length="0.030"/>
+		</geometry>
+		<material name="roller_metal"/>
+	  </visual>
+	  <visual>
+		<origin xyz="${direction * 0.080} ${side * 0.020} -0.010" rpy="1.57079632679 0 0"/>
+		<geometry>
+		  <cylinder radius="0.012" length="0.030"/>
+		</geometry>
+		<material name="roller_metal"/>
 	  </visual>
 	  <collision>
+		<origin xyz="${direction * 0.045} ${side * 0.020} -0.010"/>
 		<geometry>
-		  <!-- Keep mesh visuals, but use portable primitive collision. -->
-		  <box size="0.055 0.018 0.012"/>
+		  <box size="0.100 0.024 0.030"/>
 		</geometry>
 	  </collision>
 	  <inertial>
-		<origin xyz="0 0 -0.02"/>
+		<origin xyz="${direction * 0.045} ${side * 0.020} -0.010"/>
 		<mass value="0.15"/>
-		<inertia ixx="0.00001" ixy="0" ixz="0" iyy="0.00001" iyz="0" izz="0.000004" />
+		<inertia ixx="0.000025" ixy="0" ixz="0" iyy="0.000150" iyz="0" izz="0.000150" />
 	  </inertial>
 	</link>

File: spider_simulation/src/spider_robot_description/robots/parts/wheel/wheel.urdf.xacro (robot description, xacro)
@@ -14,9 +14,10 @@
 	</joint>
 	<link name="${prefix}_wheel_link">
-	  <visual>
-		<geometry>
-		  <mesh filename="package://spider_robot_description/meshes/DAE/wheel/wheel_link.dae"/>
-		</geometry>
-	  </visual>
+	  <!--
+	    Gazebo's DiffDrive system requires rotating wheel joints. These
+	    cylinders are deliberately collision-only: the Spider is rendered as a
+	    tracked vehicle, while the hidden contacts provide stable skid-steer
+	    physics.
+	  -->
 	  <collision>
 		<origin xyz="0 0 0" rpy="1.57079632679 0 0"/>

File: spider_simulation/src/spider_robot_description/robots/spider_robot.urdf.xacro (robot description, xacro)
@@ -15,4 +15,13 @@
     <color rgba="1.0 1.0 1.0 1.0"/>
   </material>
+  <material name="track_rubber">
+    <color rgba="0.035 0.045 0.055 1.0"/>
+  </material>
+  <material name="spider_orange">
+    <color rgba="0.95 0.32 0.04 1.0"/>
+  </material>
+  <material name="roller_metal">
+    <color rgba="0.30 0.34 0.38 1.0"/>
+  </material>
   <!-- =============== Link & Joint =============== -->
   <!-- Base -->
@@ -29,44 +38,44 @@
 	<origin xyz="0.0 0 0.035"/>
   </xacro:lidar_head_v0>
-  <!-- Suspension -->
-  <!-- Front Right Sus -->
-  <xacro:steering_v0 prefix="fr" parent="base_link">
+  <!-- Articulated tracked flippers -->
+  <!-- Front right flipper -->
+  <xacro:flipper_v0 prefix="fr" parent="base_link" direction="1" side="-1">
 	<origin xyz="0.077 -0.031 -0.004"/>
-	<axis xyz="0 0 1"/>
-  </xacro:steering_v0>
-  <!-- Front Left Sus -->
-  <xacro:steering_v0 prefix="fl" parent="base_link">
+	<axis xyz="0 -1 0"/>
+  </xacro:flipper_v0>
+  <!-- Front left flipper -->
+  <xacro:flipper_v0 prefix="fl" parent="base_link" direction="1" side="1">
 	<origin xyz="0.077 0.031 -0.004"/>
-	<axis xyz="0 0 1"/>
-  </xacro:steering_v0>
-  <!-- Rear Right Sus -->
-  <xacro:steering_v0 prefix="rr" parent="base_link">
+	<axis xyz="0 -1 0"/>
+  </xacro:flipper_v0>
+  <!-- Rear right flipper -->
+  <xacro:flipper_v0 prefix="rr" parent="base_link" direction="-1" side="-1">
 	<origin xyz="-0.077 -0.031 -0.004"/>
-	<axis xyz="0 0 1"/>
-  </xacro:steering_v0>
-  <!-- Rear Left Sus -->
-  <xacro:steering_v0 prefix="rl" parent="base_link">
+	<axis xyz="0 1 0"/>
+  </xacro:flipper_v0>
+  <!-- Rear left flipper -->
+  <xacro:flipper_v0 prefix="rl" parent="base_link" direction="-1" side="1">
 	<origin xyz="-0.077 0.031 -0.004"/>
-	<axis xyz="0 0 1"/>
-  </xacro:steering_v0>
+	<axis xyz="0 1 0"/>
+  </xacro:flipper_v0>
   <!-- Wheel -->
   <!-- Front Right Wheel -->
-  <xacro:wheel_v0 prefix="fr" parent="fr_steering_link">
-	<origin xyz="0 -0.021 -0.025"/>
+  <xacro:wheel_v0 prefix="fr" parent="base_link">
+	<origin xyz="0.077 -0.052 -0.029"/>
 	<axis xyz="0 1 0"/>
   </xacro:wheel_v0>
   <!--  Front Left Wheel -->
-  <xacro:wheel_v0 prefix="fl" parent="fl_steering_link">
-	<origin xyz="0 0.021 -0.025" rpy="0 0 ${M_PI}"/>
+  <xacro:wheel_v0 prefix="fl" parent="base_link">
+	<origin xyz="0.077 0.052 -0.029" rpy="0 0 ${M_PI}"/>
 	<axis xyz="0 -1 0"/>
   </xacro:wheel_v0>
   <!-- Rear Right Wheel -->
-  <xacro:wheel_v0 prefix="rr" parent="rr_steering_link">
-	<origin xyz="0 -0.021 -0.025"/>
+  <xacro:wheel_v0 prefix="rr" parent="base_link">
+	<origin xyz="-0.077 -0.052 -0.029"/>
 	<axis xyz="0 1 0"/>
   </xacro:wheel_v0>
   <!--  Rear Left Wheel -->
-  <xacro:wheel_v0 prefix="rl" parent="rl_steering_link">
-	<origin xyz="0 0.021 -0.025" rpy="0 0 ${M_PI}"/>
+  <xacro:wheel_v0 prefix="rl" parent="base_link">
+	<origin xyz="-0.077 0.052 -0.029" rpy="0 0 ${M_PI}"/>
 	<axis xyz="0 -1 0"/>
   </xacro:wheel_v0>
@@ -83,9 +92,9 @@
   <xacro:wheel_gazebo_v0 prefix="rr"/>
   <xacro:wheel_gazebo_v0 prefix="rl"/>
-  <!-- Steering -->
-  <xacro:steering_gazebo_v0 prefix="front_right"/>
-  <xacro:steering_gazebo_v0 prefix="front_left"/>
-  <xacro:steering_gazebo_v0 prefix="rear_right"/>
-  <xacro:steering_gazebo_v0 prefix="rear_left"/>
+  <!-- Flippers -->
+  <xacro:flipper_gazebo_v0 prefix="fr"/>
+  <xacro:flipper_gazebo_v0 prefix="fl"/>
+  <xacro:flipper_gazebo_v0 prefix="rr"/>
+  <xacro:flipper_gazebo_v0 prefix="rl"/>
   <xacro:spider_robot_gazebo/>
 </robot>

File: spider_simulation/src/spider_robot_description/ros2_control/spider_robot.ros2_control.xacro (robot description, xacro)
@@ -42,5 +42,5 @@
         <state_interface name="effort"/>
       </joint>
-      <joint name="fl_steering_joint">
+      <joint name="fl_flipper_joint">
         <command_interface name="position">
           <param name="min">-3.14</param>
@@ -51,5 +51,5 @@
         <state_interface name="effort"/>
       </joint>
-      <joint name="fr_steering_joint">
+      <joint name="fr_flipper_joint">
         <command_interface name="position">
           <param name="min">-3.14</param>
@@ -60,5 +60,5 @@
         <state_interface name="effort"/>
       </joint>
-      <joint name="rl_steering_joint">
+      <joint name="rl_flipper_joint">
         <command_interface name="position">
           <param name="min">-3.14</param>
@@ -69,5 +69,5 @@
         <state_interface name="effort"/>
       </joint>
-      <joint name="rr_steering_joint">
+      <joint name="rr_flipper_joint">
         <command_interface name="position">
           <param name="min">-3.14</param>
