Commit message: Spider has flippers

File: spider_simulation/src/spider_robot_description/gazebo/spider_robot.gazebo.xacro (robot description, xacro)
@@ -15,11 +15,17 @@
       <joint_name>${joint}</joint_name>
       <topic>${topic}</topic>
-      <p_gain>2.0</p_gain>
-      <i_gain>0.05</i_gain>
-      <d_gain>0.1</d_gain>
-      <i_max>1.0</i_max>
-      <i_min>-1.0</i_min>
-      <cmd_max>20.0</cmd_max>
-      <cmd_min>-20.0</cmd_min>
+      <!--
+        An arm holds its own 0.322 kg plus a 0.898 kg wheel at 0.24 m, so
+        gravity alone asks about 2.5 N.m at full extension. The previous
+        gains were sized for the old decorative flippers and sag under that.
+        cmd_max matches the joint's 100 N.m effort limit.
+      -->
+      <p_gain>50.0</p_gain>
+      <i_gain>1.0</i_gain>
+      <d_gain>5.0</d_gain>
+      <i_max>20.0</i_max>
+      <i_min>-20.0</i_min>
+      <cmd_max>100.0</cmd_max>
+      <cmd_min>-100.0</cmd_min>
     </plugin>
   </xacro:macro>
@@ -27,14 +33,25 @@
     <!-- =============== Gazebo =============== -->
     <gazebo>
-      <!-- Tracks: skid steer approximated as a differential drive across both
-           wheels on each side. -->
+      <!-- Tracks: skid steer approximated as a differential drive across all
+           four track wheels on each side. -->
       <plugin filename="gz-sim-diff-drive-system"
               name="gz::sim::systems::DiffDrive">
-        <left_joint>fl_wheel_joint</left_joint>
-        <left_joint>rl_wheel_joint</left_joint>
-        <right_joint>fr_wheel_joint</right_joint>
-        <right_joint>rr_wheel_joint</right_joint>
-        <wheel_separation>0.122</wheel_separation>
-        <wheel_radius>0.026</wheel_radius>
+        <left_joint>fl_track_wheel_joint</left_joint>
+        <left_joint>fl_track_wheel_2_joint</left_joint>
+        <left_joint>rl_track_wheel_joint</left_joint>
+        <left_joint>rl_track_wheel_2_joint</left_joint>
+        <right_joint>fr_track_wheel_joint</right_joint>
+        <right_joint>fr_track_wheel_2_joint</right_joint>
+        <right_joint>rr_track_wheel_joint</right_joint>
+        <right_joint>rr_track_wheel_2_joint</right_joint>
+        <!--
+          Geometric separation: the arm pivots sit at y=+/-0.0755 and each
+          wheel a further 0.06 outboard, so 2 * 0.1355. The source description
+          declared 0.3 to its ROS 1 skid-steer plugin, but that value only
+          scaled that plugin's mixing; odometry here is better served by the
+          real number.
+        -->
+        <wheel_separation>0.271</wheel_separation>
+        <wheel_radius>0.1</wheel_radius>
         <max_linear_acceleration>2.0</max_linear_acceleration>
         <topic>cmd_vel</topic>
@@ -44,5 +61,5 @@
         <odom_publish_frequency>50</odom_publish_frequency>
       </plugin>
-      <!-- Position control holds the flippers against gravity, matching the
+      <!-- Position control holds the arms against gravity, matching the
            real Teensy PID loop. -->
       <xacro:flipper_controller joint="fl_flipper_joint" topic="flipper/fl"/>

File: spider_simulation/src/spider_robot_description/robots/parts/base/base.urdf.xacro (robot description, xacro)
@@ -2,35 +2,13 @@
 <robot xmlns:xacro="http://ros.org/wiki/xacro">
   <xacro:include filename="$(find spider_robot_description)/robots/parts/base/base.gazebo.xacro"/>
-  <xacro:macro name="main_track_visual" params="side">
-	<!-- Fixed visible track; hidden wheel contacts supply its motion. -->
-	<visual>
-	  <origin xyz="0 ${side * 0.052} -0.010"/>
-	  <geometry>
-		<box size="0.145 0.030 0.047"/>
-	  </geometry>
-	  <material name="track_rubber"/>
-	</visual>
-	<visual>
-	  <origin xyz="0 ${side * 0.052} -0.010"/>
-	  <geometry>
-		<box size="0.108 0.033 0.027"/>
-	  </geometry>
-	  <material name="spider_orange"/>
-	</visual>
-	<visual>
-	  <origin xyz="0.050 ${side * 0.052} -0.010" rpy="1.57079632679 0 0"/>
-	  <geometry>
-		<cylinder radius="0.017" length="0.035"/>
-	  </geometry>
-	  <material name="roller_metal"/>
-	</visual>
-	<visual>
-	  <origin xyz="-0.050 ${side * 0.052} -0.010" rpy="1.57079632679 0 0"/>
-	  <geometry>
-		<cylinder radius="0.017" length="0.035"/>
-	  </geometry>
-	  <material name="roller_metal"/>
-	</visual>
-  </xacro:macro>
+  <!--
+    Spider chassis. The caller supplies the 0.1346 m lift from base_footprint
+    that the source description expressed as a separate base_link -> body_link
+    joint; folding it into this joint keeps the link names the driver and
+    DiffDrive expect.
+    Unlike the earlier version of this base, the link carries no track
+    visuals: the tracks are the flipper arms themselves, so the drive geometry
+    lives entirely in the flipper and wheel macros.
+  -->
   <xacro:macro name="base_v0" params="parent *joint_origin">
 	<joint name="base_link_joint" type="fixed">
@@ -41,21 +19,23 @@
 	<link name="base_link">
 	  <visual>
+		<origin xyz="0 0 0" rpy="0 0 0"/>
 		<geometry>
-		  <mesh filename="package://spider_robot_description/meshes/DAE/base/base_link.dae"/>
+		  <mesh filename="package://spider_robot_description/meshes/STL/spider/Body_bin.STL"
+		        scale="0.001 0.001 0.001"/>
 		</geometry>
+		<material name="spider_gray"/>
 	  </visual>
-	  <xacro:main_track_visual side="1"/>
-	  <xacro:main_track_visual side="-1"/>
 	  <collision>
-		<origin xyz="0 0 0.017"/>
+		<origin xyz="0 0 0" rpy="0 0 0"/>
 		<geometry>
-		  <!-- DART cannot create collision shapes from the original STL. -->
-		  <box size="0.19 0.09 0.034"/>
+		  <!-- Primitive collision; DART cannot build a shape from the mesh. -->
+		  <box size="0.293 0.190 0.073"/>
 		</geometry>
 	  </collision>
 	  <inertial>
-		<origin xyz="0 0 0.017"/>
-		<mass value="1.2"/>
-		<inertia ixx="0.0001873" ixy="0" ixz="0" iyy="0.000055" iyz="0" izz="0.0002283" />
+		<origin xyz="0 0 0.003" rpy="0 0 0"/>
+		<mass value="0.843"/>
+		<inertia ixx="0.004376981" ixy="0" ixz="0"
+		         iyy="0.010878840" iyz="0" izz="0.014340315"/>
 	  </inertial>
 	</link>

File: spider_simulation/src/spider_robot_description/robots/parts/suspension/suspension.urdf.xacro (robot description, xacro)
@@ -2,54 +2,60 @@
 <robot xmlns:xacro="http://ros.org/wiki/xacro">
   <xacro:include filename="$(find spider_robot_description)/robots/parts/suspension/suspension.gazebo.xacro"/>
-  <xacro:macro name="flipper_v0" params="prefix parent direction side *joint_origin *joint_axis">
+  <!--
+    Spider flipper arm. On this robot the flipper is not decoration: it is the
+    track frame, and it carries the two wheels its track runs around (see
+    wheel.urdf.xacro). Rotating the joint swings the outer wheel up, which is
+    what lets the vehicle climb.
+    Two mirrored meshes are supplied (FL/RR share one, FR/RL the other) and the
+    inertial and collision offsets flip sign with them, so both are derived
+    from the mesh name rather than passed separately.
+  -->
+  <xacro:property name="flipper_stl_1" value="Flipper_FL_RR_bin.STL"/>
+  <xacro:property name="flipper_stl_2" value="Flipper_FR_RL_bin.STL"/>
+  <xacro:macro name="flipper_v0" params="prefix parent stl *joint_origin *joint_axis">
 	<joint name="${prefix}_flipper_joint" type="revolute">
 	  <xacro:insert_block name="joint_origin"/>
 	  <parent link="${parent}"/>
 	  <child link="${prefix}_flipper_link"/>
-          <limit effort="5" velocity="6.28"  lower="-2.1" upper="2.1" />
-          <xacro:insert_block name="joint_axis"/>
+	  <xacro:insert_block name="joint_axis"/>
+	  <dynamics damping="0.001" friction="0.0001"/>
+	  <!--
+	    The source description declares these joints "continuous" yet gives them
+	    limits, which URDF ignores on a continuous joint. Declaring them
+	    revolute makes the limits real, which the gz JointPositionController
+	    and the driver's own clamp both rely on. 1.46 rad = 83.6 deg.
+	  -->
+	  <limit effort="100" velocity="1.5708" lower="-1.46" upper="1.46"/>
 	</joint>
 	<link name="${prefix}_flipper_link">
-	  <!-- Rubber belt around the flipper body. -->
 	  <visual>
-		<origin xyz="${direction * 0.045} ${side * 0.020} -0.010"/>
+		<origin xyz="0 0 0" rpy="0 0 0"/>
 		<geometry>
-		  <box size="0.105 0.026 0.034"/>
+		  <mesh filename="package://spider_robot_description/meshes/STL/spider/${stl}"
+		        scale="0.001 0.001 0.001"/>
 		</geometry>
-		<material name="track_rubber"/>
-	  </visual>
-	  <!-- Coloured side plate leaves a dark belt visible around its edge. -->
-	  <visual>
-		<origin xyz="${direction * 0.045} ${side * 0.020} -0.010"/>
-		<geometry>
-		  <box size="0.077 0.029 0.018"/>
-		</geometry>
-		<material name="spider_orange"/>
-	  </visual>
-	  <!-- End rollers make the primitive geometry read as a tracked flipper. -->
-	  <visual>
-		<origin xyz="${direction * 0.010} ${side * 0.020} -0.010" rpy="1.57079632679 0 0"/>
-		<geometry>
-		  <cylinder radius="0.012" length="0.030"/>
-		</geometry>
-		<material name="roller_metal"/>
-	  </visual>
-	  <visual>
-		<origin xyz="${direction * 0.080} ${side * 0.020} -0.010" rpy="1.57079632679 0 0"/>
-		<geometry>
-		  <cylinder radius="0.012" length="0.030"/>
-		</geometry>
-		<material name="roller_metal"/>
+		<material name="spider_black"/>
 	  </visual>
 	  <collision>
-		<origin xyz="${direction * 0.045} ${side * 0.020} -0.010"/>
+		<xacro:if value="${stl == flipper_stl_1}">
+		  <origin xyz="0.119 0.021 0.035" rpy="0 0 0"/>
+		</xacro:if>
+		<xacro:unless value="${stl == flipper_stl_1}">
+		  <origin xyz="0.119 -0.021 0.034" rpy="0 0 0"/>
+		</xacro:unless>
 		<geometry>
-		  <box size="0.100 0.024 0.030"/>
+		  <box size="0.316 0.091 0.146"/>
 		</geometry>
 	  </collision>
 	  <inertial>
-		<origin xyz="${direction * 0.045} ${side * 0.020} -0.010"/>
-		<mass value="0.15"/>
-		<inertia ixx="0.000025" ixy="0" ixz="0" iyy="0.000150" iyz="0" izz="0.000150" />
+		<xacro:if value="${stl == flipper_stl_1}">
+		  <origin xyz="0.123 0.033 0.029" rpy="0 0 0"/>
+		</xacro:if>
+		<xacro:unless value="${stl == flipper_stl_1}">
+		  <origin xyz="0.123 -0.033 0.029" rpy="0 0 0"/>
+		</xacro:unless>
+		<mass value="0.322"/>
+		<inertia ixx="0.001119686" ixy="0.0001239386" ixz="0.0001140656"
+		         iyy="0.008247686" iyz="0.000378888" izz="0.007985380"/>
 	  </inertial>
 	</link>

File: spider_simulation/src/spider_robot_description/robots/parts/wheel/wheel.gazebo.xacro (robot description, xacro)
@@ -1,6 +1,6 @@
 <?xml version="1.0"?>
 <robot xmlns:xacro="http://ros.org/wiki/xacro">
-  <xacro:macro name="wheel_gazebo_v0" params="prefix">
-    <gazebo reference="${prefix}_wheel_link">
+  <xacro:macro name="wheel_gazebo_v0" params="prefix suffix:=''">
+    <gazebo reference="${prefix}_track_wheel${suffix}_link">
       <selfCollide>false</selfCollide>
       <mu1 value="1.2" />

File: spider_simulation/src/spider_robot_description/robots/parts/wheel/wheel.urdf.xacro (robot description, xacro)
@@ -2,33 +2,63 @@
 <robot xmlns:xacro="http://ros.org/wiki/xacro">
   <xacro:include filename="$(find spider_robot_description)/robots/parts/wheel/wheel.gazebo.xacro"/>
-  <xacro:macro name="wheel_v0" params="prefix parent *joint_origin *joint_axis">
-	<joint name="${prefix}_wheel_joint" type="continuous">
+  <!--
+    A wheel that a flipper's track runs around, not a road wheel: two per
+    flipper, the inner one on the flipper's own pivot axis so it stays put as
+    the arm swings, the outer one at the arm's tip. The parent is therefore
+    the flipper link, not base_link.
+    `suffix` selects which of the pair this is. It is empty for the inner
+    wheel, whose joint the Teensy bridge reads telemetry from; the outer one
+    becomes `_track_wheel_2_`.
+    As with the flippers, the mirrored L/R meshes carry mirrored offsets, so
+    both are derived from the mesh name.
+  -->
+  <xacro:property name="wheel_stl_l" value="Wheel_L_bin.STL"/>
+  <xacro:property name="wheel_stl_r" value="Wheel_R_bin.STL"/>
+  <xacro:macro name="wheel_v0" params="prefix parent stl suffix:='' *joint_origin">
+	<joint name="${prefix}_track_wheel${suffix}_joint" type="continuous">
 	  <xacro:insert_block name="joint_origin"/>
 	  <parent link="${parent}"/>
-	  <child link="${prefix}_wheel_link"/>
-      <!-- At the 0.026 m wheel radius, a full 1 m/s + 1 rad/s TWIST needs
-           40.81 rad/s on the faster side. A 20 rad/s cap saturated both
-           sides equally at high throttle and erased the steering command. -->
-      <limit effort="1.5" velocity="50"/>
-	  <xacro:insert_block name="joint_axis"/>
+	  <child link="${prefix}_track_wheel${suffix}_link"/>
+	  <axis xyz="0 1 0"/>
+	  <!--
+	    At the 0.1 m Spider wheel radius a full 1 m/s + 1 rad/s TWIST needs
+	    about 11.4 rad/s on the faster side, so 20 rad/s leaves headroom
+	    without letting the faster side saturate and erase the steering
+	    command. Effort matches the 20 N.m the source description gave its
+	    drive plugin.
+	  -->
+	  <limit effort="20" velocity="20"/>
 	</joint>
-	<link name="${prefix}_wheel_link">
-	  <!--
-	    Gazebo's DiffDrive system requires rotating wheel joints. These
-	    cylinders are deliberately collision-only: the Spider is rendered as a
-	    tracked vehicle, while the hidden contacts provide stable skid-steer
-	    physics.
-	  -->
+	<link name="${prefix}_track_wheel${suffix}_link">
+	  <visual>
+		<origin xyz="0 0 0" rpy="0 0 0"/>
+		<geometry>
+		  <mesh filename="package://spider_robot_description/meshes/STL/spider/${stl}"
+		        scale="0.001 0.001 0.001"/>
+		</geometry>
+		<material name="spider_gray"/>
+	  </visual>
 	  <collision>
-		<origin xyz="0 0 0" rpy="1.57079632679 0 0"/>
+		<xacro:if value="${stl == wheel_stl_l}">
+		  <origin xyz="0 0.031 0" rpy="1.57079632679 0 0"/>
+		</xacro:if>
+		<xacro:unless value="${stl == wheel_stl_l}">
+		  <origin xyz="0 -0.031 0" rpy="1.57079632679 0 0"/>
+		</xacro:unless>
 		<geometry>
 		  <!-- Primitive collision works with Gazebo's default DART engine. -->
-		  <cylinder radius="0.026" length="0.020"/>
+		  <cylinder radius="0.1" length="0.11"/>
 		</geometry>
 	  </collision>
 	  <inertial>
-		<origin xyz="0.0 -0.007 -0.0"/>
-		<mass value="0.05"/>
-		<inertia ixx="0.00001" ixy="0" ixz="0" iyy="0.000018" iyz="0" izz="0.00001"/>
+		<xacro:if value="${stl == wheel_stl_l}">
+		  <origin xyz="0 0.039 0" rpy="0 0 0"/>
+		</xacro:if>
+		<xacro:unless value="${stl == wheel_stl_l}">
+		  <origin xyz="0 -0.039 0" rpy="0 0 0"/>
+		</xacro:unless>
+		<mass value="0.898"/>
+		<inertia ixx="0.003834480" ixy="0" ixz="0"
+		         iyy="0.004561738" iyz="0" izz="0.003834480"/>
 	  </inertial>
 	</link>

File: spider_simulation/src/spider_robot_description/robots/spider_robot.urdf.xacro (robot description, xacro)
@@ -1,4 +1,4 @@
 <?xml version="1.0"?>
-<!-- Basic differential drive mobile base -->
+<!-- Spider: tracked chassis on four independently articulated track arms -->
 <robot xmlns:xacro="http://www.ros.org/wiki/xacro" name="spider_robot">
   <xacro:include filename="$(find spider_robot_description)/gazebo/spider_robot.gazebo.xacro" />
@@ -9,4 +9,10 @@
   <xacro:include filename="$(find spider_robot_description)/robots/parts/lidar_head/lidar_head.urdf.xacro"/>
   <xacro:property name="M_PI" value="3.14159274"/>
+  <material name="spider_gray">
+    <color rgba="0.55 0.55 0.55 1.0"/>
+  </material>
+  <material name="spider_black">
+    <color rgba="0.15 0.15 0.15 1.0"/>
+  </material>
   <material name="gray">
     <color rgba="0.5 0.5 0.5 1.0"/>
@@ -15,86 +21,90 @@
     <color rgba="1.0 1.0 1.0 1.0"/>
   </material>
-  <material name="track_rubber">
-    <color rgba="0.035 0.045 0.055 1.0"/>
-  </material>
-  <material name="spider_orange">
-    <color rgba="0.95 0.32 0.04 1.0"/>
-  </material>
-  <material name="roller_metal">
-    <color rgba="0.30 0.34 0.38 1.0"/>
-  </material>
   <!-- =============== Link & Joint =============== -->
-  <!-- Base -->
-  <link name="base_footprint"/> <!--link name="base_footprint"/ -->
-  <xacro:base_v0 parent="base_footprint"> <!-- xacro:base_v0 parent="base_footprint" -->
-	<origin xyz="0 0 0"/>
+  <!--
+    Base. The source description lifts the chassis 0.1346 m over the
+    ground-level root through a separate body_link; that offset is folded into
+    base_link_joint here so the link names stay the ones DiffDrive and the
+    Teensy bridge already use.
+  -->
+  <link name="base_footprint"/>
+  <xacro:base_v0 parent="base_footprint">
+	<origin xyz="0 0 0.1346"/>
   </xacro:base_v0>
-  <!-- lidar_base -->
+  <!-- lidar_base: 0.0365 clears the top face of the 0.073 m chassis -->
   <xacro:lidar_base_v0 parent="base_link">
-	<origin xyz="-0.022 0 0.035"/>
+	<origin xyz="-0.022 0 0.037"/>
   </xacro:lidar_base_v0>
   <!-- lidar_head -->
   <xacro:lidar_head_v0 parent="base_link">
-	<origin xyz="0.0 0 0.035"/>
+	<origin xyz="0.0 0 0.037"/>
   </xacro:lidar_head_v0>
-  <!-- Articulated tracked flippers -->
-  <!-- Front right flipper -->
-  <xacro:flipper_v0 prefix="fr" parent="base_link" direction="1" side="-1">
-	<origin xyz="0.077 -0.031 -0.004"/>
+  <!--
+    Track arms. The rear pair is yawed by pi so the arm extends rearwards; that
+    is also why its joint axis is negated, keeping a positive command "arm up"
+    on all four corners.
+  -->
+  <xacro:flipper_v0 prefix="fl" parent="base_link" stl="${flipper_stl_1}">
+	<origin xyz="0.115 0.0755 -0.005" rpy="0 0 0"/>
+	<axis xyz="0 1 0"/>
+  </xacro:flipper_v0>
+  <xacro:flipper_v0 prefix="fr" parent="base_link" stl="${flipper_stl_2}">
+	<origin xyz="0.115 -0.0755 -0.005" rpy="0 0 0"/>
+	<axis xyz="0 1 0"/>
+  </xacro:flipper_v0>
+  <xacro:flipper_v0 prefix="rl" parent="base_link" stl="${flipper_stl_2}">
+	<origin xyz="-0.115 0.0755 -0.005" rpy="0 0 ${M_PI}"/>
 	<axis xyz="0 -1 0"/>
   </xacro:flipper_v0>
-  <!-- Front left flipper -->
-  <xacro:flipper_v0 prefix="fl" parent="base_link" direction="1" side="1">
-	<origin xyz="0.077 0.031 -0.004"/>
+  <xacro:flipper_v0 prefix="rr" parent="base_link" stl="${flipper_stl_1}">
+	<origin xyz="-0.115 -0.0755 -0.005" rpy="0 0 ${M_PI}"/>
 	<axis xyz="0 -1 0"/>
   </xacro:flipper_v0>
-  <!-- Rear right flipper -->
-  <xacro:flipper_v0 prefix="rr" parent="base_link" direction="-1" side="-1">
-	<origin xyz="-0.077 -0.031 -0.004"/>
-	<axis xyz="0 1 0"/>
-  </xacro:flipper_v0>
-  <!-- Rear left flipper -->
-  <xacro:flipper_v0 prefix="rl" parent="base_link" direction="-1" side="1">
-	<origin xyz="-0.077 0.031 -0.004"/>
-	<axis xyz="0 1 0"/>
-  </xacro:flipper_v0>
-  <!-- Wheel -->
-  <!-- Front Right Wheel -->
-  <xacro:wheel_v0 prefix="fr" parent="base_link">
-	<origin xyz="0.077 -0.052 -0.029"/>
-	<axis xyz="0 1 0"/>
+  <!--
+    Track wheels, two per flipper. The inner one sits on the arm's pivot axis
+    (x=0) and keeps the unsuffixed joint name; the outer one rides at x=0.24.
+    The rear joints carry a second yaw of pi which cancels the arm's own, so
+    every track wheel still spins about body +y.
+  -->
+  <xacro:wheel_v0 prefix="fl" parent="fl_flipper_link" stl="${wheel_stl_l}">
+	<origin xyz="0 0.06 0" rpy="0 0 0"/>
   </xacro:wheel_v0>
-  <!--  Front Left Wheel -->
-  <xacro:wheel_v0 prefix="fl" parent="base_link">
-	<origin xyz="0.077 0.052 -0.029" rpy="0 0 ${M_PI}"/>
-	<axis xyz="0 -1 0"/>
+  <xacro:wheel_v0 prefix="fl" parent="fl_flipper_link" stl="${wheel_stl_l}" suffix="_2">
+	<origin xyz="0.24 0.06 0" rpy="0 0 0"/>
   </xacro:wheel_v0>
-  <!-- Rear Right Wheel -->
-  <xacro:wheel_v0 prefix="rr" parent="base_link">
-	<origin xyz="-0.077 -0.052 -0.029"/>
-	<axis xyz="0 1 0"/>
+  <xacro:wheel_v0 prefix="fr" parent="fr_flipper_link" stl="${wheel_stl_r}">
+	<origin xyz="0 -0.06 0" rpy="0 0 0"/>
   </xacro:wheel_v0>
-  <!--  Rear Left Wheel -->
-  <xacro:wheel_v0 prefix="rl" parent="base_link">
-	<origin xyz="-0.077 0.052 -0.029" rpy="0 0 ${M_PI}"/>
-	<axis xyz="0 -1 0"/>
+  <xacro:wheel_v0 prefix="fr" parent="fr_flipper_link" stl="${wheel_stl_r}" suffix="_2">
+	<origin xyz="0.24 -0.06 0" rpy="0 0 0"/>
+  </xacro:wheel_v0>
+  <xacro:wheel_v0 prefix="rl" parent="rl_flipper_link" stl="${wheel_stl_l}">
+	<origin xyz="0 -0.06 0" rpy="0 0 ${M_PI}"/>
+  </xacro:wheel_v0>
+  <xacro:wheel_v0 prefix="rl" parent="rl_flipper_link" stl="${wheel_stl_l}" suffix="_2">
+	<origin xyz="0.24 -0.06 0" rpy="0 0 ${M_PI}"/>
+  </xacro:wheel_v0>
+  <xacro:wheel_v0 prefix="rr" parent="rr_flipper_link" stl="${wheel_stl_r}">
+	<origin xyz="0 0.06 0" rpy="0 0 ${M_PI}"/>
+  </xacro:wheel_v0>
+  <xacro:wheel_v0 prefix="rr" parent="rr_flipper_link" stl="${wheel_stl_r}" suffix="_2">
+	<origin xyz="0.24 0.06 0" rpy="0 0 ${M_PI}"/>
   </xacro:wheel_v0>
   <!-- =============== Gazebo =============== -->
-  <!-- Base -->
   <xacro:base_gazebo_v0/>
-  <!-- lidar base -->
   <xacro:lidar_base_gazebo_v0/>
-  <!-- lidar head -->
   <xacro:lidar_head_gazebo_v0/>
-  <!-- Wheel -->
+  <xacro:wheel_gazebo_v0 prefix="fl"/>
   <xacro:wheel_gazebo_v0 prefix="fr"/>
-  <xacro:wheel_gazebo_v0 prefix="fl"/>
+  <xacro:wheel_gazebo_v0 prefix="rl"/>
   <xacro:wheel_gazebo_v0 prefix="rr"/>
-  <xacro:wheel_gazebo_v0 prefix="rl"/>
-  <!-- Flippers -->
+  <xacro:wheel_gazebo_v0 prefix="fl" suffix="_2"/>
+  <xacro:wheel_gazebo_v0 prefix="fr" suffix="_2"/>
+  <xacro:wheel_gazebo_v0 prefix="rl" suffix="_2"/>
+  <xacro:wheel_gazebo_v0 prefix="rr" suffix="_2"/>
+  <xacro:flipper_gazebo_v0 prefix="fl"/>
   <xacro:flipper_gazebo_v0 prefix="fr"/>
-  <xacro:flipper_gazebo_v0 prefix="fl"/>
+  <xacro:flipper_gazebo_v0 prefix="rl"/>
   <xacro:flipper_gazebo_v0 prefix="rr"/>
-  <xacro:flipper_gazebo_v0 prefix="rl"/>
   <xacro:spider_robot_gazebo/>
 </robot>
