Commit message: Spider has flippers

File: spider_simulation/src/spider_robot_description/ros2_control/spider_robot.ros2_control.xacro (robot description, xacro)
@@ -6,5 +6,5 @@
           <plugin>gz_ros2_control/GazeboSimSystem</plugin>
       </hardware>
-      <joint name="fl_wheel_joint">
+      <joint name="fl_track_wheel_joint">
         <command_interface name="velocity">
           <param name="min">-1</param>
@@ -15,5 +15,5 @@
         <state_interface name="effort"/>
       </joint>
-      <joint name="fr_wheel_joint">
+      <joint name="fl_track_wheel_2_joint">
         <command_interface name="velocity">
           <param name="min">-1</param>
@@ -24,5 +24,5 @@
         <state_interface name="effort"/>
       </joint>
-      <joint name="rl_wheel_joint">
+      <joint name="fr_track_wheel_joint">
         <command_interface name="velocity">
           <param name="min">-1</param>
@@ -33,5 +33,41 @@
         <state_interface name="effort"/>
       </joint>
-      <joint name="rr_wheel_joint">
+      <joint name="fr_track_wheel_2_joint">
+        <command_interface name="velocity">
+          <param name="min">-1</param>
+          <param name="max">1</param>
+        </command_interface>
+        <state_interface name="position"/>
+        <state_interface name="velocity"/>
+        <state_interface name="effort"/>
+      </joint>
+      <joint name="rl_track_wheel_joint">
+        <command_interface name="velocity">
+          <param name="min">-1</param>
+          <param name="max">1</param>
+        </command_interface>
+        <state_interface name="position"/>
+        <state_interface name="velocity"/>
+        <state_interface name="effort"/>
+      </joint>
+      <joint name="rl_track_wheel_2_joint">
+        <command_interface name="velocity">
+          <param name="min">-1</param>
+          <param name="max">1</param>
+        </command_interface>
+        <state_interface name="position"/>
+        <state_interface name="velocity"/>
+        <state_interface name="effort"/>
+      </joint>
+      <joint name="rr_track_wheel_joint">
+        <command_interface name="velocity">
+          <param name="min">-1</param>
+          <param name="max">1</param>
+        </command_interface>
+        <state_interface name="position"/>
+        <state_interface name="velocity"/>
+        <state_interface name="effort"/>
+      </joint>
+      <joint name="rr_track_wheel_2_joint">
         <command_interface name="velocity">
           <param name="min">-1</param>
